File: KICAD GIT/TestGithub/TestGithub.kicad_sch (KiCad schematic)
At the start: 4 parts, among them U1 4011, U2 STM32C011F4Px, U3 STM32C011F4Px, U4 STM32C011F_4-6_Px

Commit message: Segundo commit xd
Parts:
- added J1: USB4105-GF-A, USB4105-GF-A:GCT_USB4105-GF-A, symbol USB_TYPEC:USB4105-GF-A
Changed lines of the file:
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@@
+	)
+	(symbol
+		(lib_id "USB_TYPEC:USB4105-GF-A")
+		(at 203.2 121.92 0)
+		(unit 1)
+		(exclude_from_sim no)
+		(in_bom yes)
+		(on_board yes)
+		(dnp no)
+		(fields_autoplaced yes)
+		(property "Reference" "J1"
+			(at 203.2 104.14 0)
+			(effects
+				(font
+					(size 1.27 1.27)
+				)
+			)
+		)
+		(property "Value" "USB4105-GF-A"
+			(at 203.2 106.68 0)
+			(effects
+				(font
+					(size 1.27 1.27)
+				)
+			)
+		)
+		(property "Footprint" "USB4105-GF-A:GCT_USB4105-GF-A"
+			(at 203.2 121.92 0)
+			(effects
+				(font
+					(size 1.27 1.27)
+				)
+				(justify bottom)
+				(hide yes)
+			)
+		)
+		(property "Datasheet" ""
+			(at 203.2 121.92 0)
+			(effects
+				(font
+					(size 1.27 1.27)
+				)
+				(hide yes)
+			)
+		)
+		(property "Description" ""
+			(at 203.2 121.92 0)
+			(effects
+				(font
+					(size 1.27 1.27)
+				)
+				(hide yes)
+			)
+		)
+		(property "PARTREV" "B4"
+			(at 203.2 121.92 0)
+			(effects
+				(font
+					(size 1.27 1.27)
+				)
+				(justify bottom)
+				(hide yes)
+			)
+		)
+		(property "STANDARD" "Manufacturer Recommendations"
+			(at 203.2 121.92 0)
+			(effects
+				(font
+					(size 1.27 1.27)
+				)
+				(justify bottom)
+				(hide yes)
+			)
+		)
+		(property "MAXIMUM_PACKAGE_HEIGHT" "3.31 mm"
+			(at 203.2 121.92 0)
+			(effects
+				(font
+					(size 1.27 1.27)
+				)
+				(justify bottom)
+				(hide yes)
+			)
+		)
+		(property "MANUFACTURER" "GCT"
+			(at 203.2 121.92 0)
+			(effects
+				(font
+					(size 1.27 1.27)
+				)
+				(justify bottom)
+				(hide yes)
+			)
+		)
+		(pin "A4_B9"
+		)
+		(pin "A6"
+		)
+		(pin "B4_A9"
+		)
+		(pin "SH3"
+		)
+		(pin "A7"
+		)
+		(pin "SH1"
+		)
+		(pin "SH4"
+		)
+		(pin "SH2"
+		)
+		(pin "A1_B12"
+		)
+		(pin "B8"
+		)
+		(pin "A5"
+		)
+		(pin "B6"
+		)
+		(pin "B1_A12"
+		)
+		(pin "B5"
+		)
+		(pin "B7"
+		)
+		(pin "A8"
+		)
+		(instances
+			(project ""
+				(path "/7c1bafac-376f-46e2-b0e2-1f7431634887"
+					(reference "J1")
+					(unit 1)
+				)
+			)
+		)
 	)
 	(symbol
